Commit message: arm :)

File: PC_user/src/Hardware/Arm/pincher_arm_description/urdf/pincher_arm.urdf.xacro (robot description, xacro)
@@ -1,6 +1,7 @@
 <?xml version="1.0"?>
 <robot name="pincher_arm" xmlns:xacro="http://ros.org/wiki/xacro">
-  <!--xacro:include filename="$(find pincher_arm_description)/urdf/pincher_arm.xacro"/-->
-  <xacro:include filename="$(find pincher_arm_description)/urdf/dark_arm.xacro"/>
+  <xacro:include filename="$(find pincher_arm_description)/urdf/robotino_kinect_arm.xacro"/>
+  <!--xacro:include filename="$(find pincher_arm_description)/urdf/dark_arm.xacro"/-->
+  <!--xacro:include filename="$(find robotino_description)/robotino_kinect.xacro"/-->
   <xacro:pincher_arm/>
 </robot>

File: PC_user/src/Hardware/Arm/pincher_arm_description/urdf/robotino_kinect_arm.xacro (robot description, xacro)
@@ -1,128 +1,136 @@
 <?xml version="1.0"?>
-<robot name="justina" xmlns:xacro="http://www.ros.org/wiki/xacro">
-	<xacro:include filename="$(find knowledge)/hardware/justina.gazebo" />
-	<!-- Import Rviz colors -->
-	<xacro:include filename="$(find knowledge)/hardware/materials.xacro" />
-	<xacro:include filename="$(find knowledge)/hardware/macros.xacro" />
-	<xacro:include filename="$(find pincher_arm_description)/urdf/arm_hardware.xacro"/>
-	<material name="White">
-    	<color rgba="0.87 0.90 0.87 1.0"/>
-  	</material>
-  	<material name="Black">
-    	<color rgba="0.08 0.08 0.08 1.0"/>
-  	</material>
-  	<material name="Gray">
-    	<color rgba="0.2 0.2 0.21 1.0"/>
-  	</material>
-  	<material name="Green">
-    	<color rgba="0.22 0.32 0.14 1.0"/>
-  	</material>
-	<xacro:property name="base_radius" value="0.21"/>
-	<xacro:property name="base_height" value="0.2156"/>
-	<xacro:property name="base_mass" value="2.0"/>
-	<xacro:property name="wheel_radius" value="0.075"/>
-	<xacro:property name="wheel_height" value="0.04"/>
-	<xacro:property name="wheel_mass" value="0.52098"/>
-	<link name="base_link"/>
-	<joint name="hex_base_connect" type="fixed">
-		<origin xyz="0 0 0" rpy="0 0 0" />
-		<parent link="base_link"/>
-		<child link="hex_base_link" />
-	</joint>
-	<link name="hex_base_link">
-		<visual>
-			<origin xyz="0.0 0.0 0.075" rpy="0.0 0 1.5708"/>
-			<!-- origin xyz="0 0 0.1828" rpy="0 0 0"/ -->
-			<geometry>
-				<mesh filename="package://knowledge/hardware/stl/base/baseHex.dae"/>
-				<!-- cylinder length="${base_height}" radius="${base_radius}"/ -->
-			</geometry>
-			<material name="grey"/>
-		</visual>
-		<collision>
-			<origin xyz="0 0 0.1828" rpy="0 0 0"/>
-			<geometry><cylinder length="${base_height}" radius="${base_radius}"/></geometry>
-		</collision>
-		<inertial>
-			<origin xyz="0 0 0.1828" rpy="0 0 0"/>
-			<mass value="${base_mass}"/>
-			<xacro:cylinder_inertia m="${base_mass}" r="${base_radius}" h="${base_height}"/>
-		</inertial>
-	</link>
-	<joint name="wheel_front_left_connect" type="continuous">
-		<origin xyz="0.1091 0.189 0.075" rpy="1.57078 0 -3.67"/>
-		<parent link="hex_base_link"/>
-		<child link="wheel_front_left"/>
-		<axis xyz="0 0 1"/>
-	</joint>
-	<link name="wheel_front_left">
-		<visual>
-			<origin xyz="0 0 0" rpy="0 3.1416 0"/>
-			<geometry>
-				<mesh filename="package://knowledge/hardware/stl/base/rueda.dae"/>
-				<!-- cylinder length="${wheel_height}" radius="${wheel_radius}"/ -->
-			</geometry>
-			<material name="grey"/>
-		</visual>
-		<collision>
-			<origin xyz="0 0 0" rpy="0 0 0"/>
-			<geometry><cylinder length="${wheel_height}" radius="${wheel_radius}"/></geometry>
-		</collision>
-		<inertial>
-			<origin xyz="0 0 0"/>
-			<mass value="${wheel_mass}"/>
-			<xacro:cylinder_inertia m="${wheel_mass}" r="${wheel_radius}" h="${wheel_height}"/>
-		</inertial>
-	</link>
-	<joint name="wheel_back_connect" type="continuous">
-		<origin xyz="-0.2182 0 0.075" rpy="1.57078 0 -1.5708"/>
-		<parent link="hex_base_link"/>
-		<child link="wheel_back"/>
-		<axis xyz="0 0 1"/>
-	</joint>
-	<link name="wheel_back">
-		<visual>
-			<origin xyz="0 0 0" rpy="0 3.1416 0"/>
-			<geometry>
-				<mesh filename="package://knowledge/hardware/stl/base/rueda.dae"/>
-				<!-- cylinder length="${wheel_height}" radius="${wheel_radius}"/ -->
-			</geometry>
-			<material name="grey"/>
-		</visual>
-		<collision>
-			<origin xyz="0 0 0" rpy="0 0 0"/>
-			<geometry><cylinder length="${wheel_height}" radius="${wheel_radius}"/></geometry>
-		</collision>
-		<inertial>
-			<origin xyz="0 0 0" rpy="0 0 0"/>
-			<mass value="${wheel_mass}"/>
-			<xacro:cylinder_inertia m="${wheel_mass}" r="${wheel_radius}" h="${wheel_height}"/>
-		</inertial>
-	</link>
-	<joint name="wheel_front_right_connect" type="continuous">
-		<origin xyz="0.1091 -0.189 0.075" rpy="1.57078 0 3.67"/>
-		<parent link="hex_base_link"/>
-		<child link="wheel_front_right"/>
-		<axis xyz="0 0 1"/>
-	</joint>
-	<link name="wheel_front_right">
-		<visual>
-			<origin xyz="0 0 0" rpy="0 0 0"/>
-			<geometry>
-				<mesh filename="package://knowledge/hardware/stl/base/rueda.dae"/>
-				<!-- cylinder length="${wheel_height}" radius="${wheel_radius}"/ -->
-			</geometry>
-			<material name="grey"/>
-		</visual>
-		<collision>
-			<origin xyz="0 0 0" rpy="0 0 0"/>
-			<geometry><cylinder length="${wheel_height}" radius="${wheel_radius}"/></geometry>
-		</collision>
-		<inertial>
-			<origin xyz="0 0 0" rpy="0 0 0"/>
-			<mass value="${wheel_mass}"/>
-			<xacro:cylinder_inertia m="${wheel_mass}" r="${wheel_radius}" h="${wheel_height}"/>
-		</inertial>
-	</link>
+<robot name="robotino" xmlns:xacro="http://www.ros.org/wiki/xacro">
+<xacro:include filename="$(find pincher_arm_description)/urdf/arm_hardware.xacro"/>
+<!-- ***************************** Main Body ***************************** -->
+  <link name="base_link">
+    <visual>
+      <origin xyz="0 0 0.035" rpy="0 0 1.5707"/>
+      <geometry>
+        <mesh filename="package://robotino_description/model/Robotino3_SplitMain.dae" scale="0.01 0.01 0.01"/>
+      </geometry>
+    </visual>
+    <collision>
+      <origin xyz="0 0 0.035" rpy="0 0 1.5707"/>
+      <geometry>
+        <mesh filename="package://robotino_description/model/Robotino3_SplitMain.dae" scale="0.01 0.01 0.01"/>
+      </geometry>
+    </collision>
+  </link>
+<!-- ***************************** Wheel 0 - Mesh ***************************** -->
+  <link name="wheel0_link">
+    <visual>
+      <origin xyz="0 0 0" rpy="0 0 0"/>
+      <geometry>
+        <mesh filename="package://robotino_description/model/Robotino3_SplitWheel.dae" scale="0.01 0.01 0.01"/>
+      </geometry>
+    </visual>
+    <collision>
+      <geometry>
+        <mesh filename="package://robotino_description/model/Robotino3_SplitWheel.dae" scale="0.01 0.01 0.01"/>
+      </geometry>
+    </collision>
+  </link>
+<!-- ========== Wheel 0 - Joint ========== -->
+  <joint name="wheel0_joint" type="continuous">
+    <parent link="base_link"/>
+    <child link="wheel0_link"/>
+    <origin xyz="-0.0001 0.1825 0.059154" rpy="0 0 0"/>
+    <axis xyz="0 1 0" rpy="0 0 0"/>
+  </joint>
+<!-- ***************************** Wheel 1 - Mesh ***************************** -->
+  <link name="wheel1_link">
+    <visual>
+      <origin xyz="0 0 0" rpy="0 0 0"/>
+      <geometry>
+        <mesh filename="package://robotino_description/model/Robotino3_SplitWheel.dae" scale="0.01 0.01 0.01"/>
+      </geometry>
+    </visual>
+    <collision>
+      <geometry>
+        <mesh filename="package://robotino_description/model/Robotino3_SplitWheel.dae" scale="0.01 0.01 0.01"/>
+      </geometry>
+    </collision>
+  </link>
+<!-- ========== Wheel 1 - Joint ========== -->
+  <joint name="wheel1_joint" type="continuous">
+    <parent link="base_link"/>
+    <child link="wheel1_link"/>
+    <origin xyz="-0.157067 -0.090625 0.059154" rpy="0 0 2.094395102393195"/>
+    <axis xyz="0 1 0" rpy="0 0 0"/>
+  </joint>
+<!-- ***************************** Wheel 2 - Mesh ***************************** -->
+  <link name="wheel2_link">
+    <visual>
+      <origin xyz="0 0 0" rpy="0 0 0"/>
+      <geometry>
+        <mesh filename="package://robotino_description/model/Robotino3_SplitWheel.dae" scale="0.01 0.01 0.01"/>
+      </geometry>
+    </visual>
+    <collision>
+      <geometry>
+        <mesh filename="package://robotino_description/model/Robotino3_SplitWheel.dae" scale="0.01 0.01 0.01"/>
+      </geometry>
+    </collision>
+  </link>
+<!-- ========== Wheel 2 - Joint ========== -->
+  <joint name="wheel2_joint" type="continuous">
+    <parent link="base_link"/>
+    <child link="wheel2_link"/>
+    <origin xyz="0.156867 -0.090625 0.059154" rpy="0 0 -2.094395102393195"/>
+    <axis xyz="0 1 0" rpy="0 0 0"/>
+  </joint>
+<!-- ***************************** Platform ***************************** -->
+<!-- Un/Comment from here to END to add/remove the platform -->
+  <link name="platform_link">
+    <visual>
+      <origin xyz="0 0 0" rpy="0 0 0"/>
+      <geometry>
+        <mesh filename="package://robotino_description/model/Robotino3_Platform.dae" scale="0.009 0.009 0.009"/>
+      </geometry>
+    </visual>
+    <collision>
+      <geometry>
+        <mesh filename="package://robotino_description/model/Robotino3_Platform.dae" scale="0.009 0.009 0.009"/>
+      </geometry>
+    </collision>
+  </link>
+<!-- ========== Platform - Joint ========== -->
+  <joint name="platform_joint" type="fixed">
+    <parent link="base_link"/>
+    <child link="platform_link"/>
+    <origin xyz="0 0 0" rpy="0 0 0"/>
+    <axis xyz="0 0 0" rpy="0 0 0"/>
+  </joint>
+<!-- ***************************** END ***************************** -->
+<!--Hokuyo :P -->
+  <link name="hokuyo_laser_link">
+    <visual>
+      <geometry>
+        <box size="0.05 0.05 0.05"/>
+      </geometry>
+      <origin xyz="0 0 0" rpy="0 0 0"/>
+    </visual>
+  </link>
+  <joint name="base_to_hokuyo" type="fixed">
+    <parent link="base_link"/>
+    <child link="hokuyo_laser_link"/>
+    <origin rpy="0 0 0" xyz="0.127 0.0 0.22"/>
+  </joint>
+<!-- Kinect o stereo camera-->
+  <link name="camera_link">
+    <visual>
+      <geometry>
+        <box size="0.03 0.14 0.0175"/>
+      </geometry>
+      <origin xyz="0 0 0" rpy="0 0 0"/>
+    </visual>
+  </link>
+ <joint name="base_to_kinect" type="fixed">
+    <parent link="base_link"/>
+    <child link="camera_link"/>
+    <!--origin rpy="0 0 0" xyz="0.13 0.0 0.91"/-->
+    <origin rpy="0 0 0" xyz="-0.07 0.0 1.22"/>
+  </joint>
+<!-- ************Arm************ -->
 <xacro:macro name="pincher_arm" params="
       color:=Gray
