Commit message: Al fiiiiiiiiiiin :) :) :) :)

File: PC_user/src/Hardware/Arm/pincher_arm_description/urdf/pincher_arm.urdf.xacro (robot description, xacro)
@@ -3,5 +3,5 @@
   <xacro:include filename="$(find pincher_arm_description)/urdf/robotino_kinect_arm.xacro"/>
   <!--xacro:include filename="$(find pincher_arm_description)/urdf/dark_arm.xacro"/-->
-  <!--xacro:include filename="$(find robotino_description)/robotino_kinect.xacro"/-->
+  <!--xacro:include filename="$(find robotino_description)/robotino_kinect_arm.xacro"/-->
   <xacro:pincher_arm/>
 </robot>

File: PC_user/src/Hardware/Robotino_pkgs/robotino_description/robotino_kinect_arm.xacro (robot description, xacro)
@@ -1,4 +1,5 @@
 <?xml version="1.0"?>
 <robot name="robotino">
+  <xacro:include filename="$(find pincher_arm_description)/urdf/arm_hardware.xacro"/>
 <!-- ***************************** Main Body ***************************** -->
   <link name="base_link">
@@ -132,694 +133,263 @@
   </joint>
 <!-- ************Arm************ -->
-<!--xacro:include filename="../arm_description/pincher_arm.urdf.xacro "-->
-<link name="arm_base_link">
-    <visual>
-      <geometry>
-        <box size="0.05 0.02 0.04"/>
-      </geometry>
-      <origin xyz="0 0 0" rpy="0 0 0"/>
-    </visual>
-  </link>
- <joint name="base_to_arm" type="fixed">
-    <parent link="base_link"/>
-    <child link="arm_base_link"/>
-    <origin rpy="0 0 0" xyz="0.15 0.0 0.97"/>
-  </joint>
-<!-- 300 degrees -->
-  <material name="White">
-    <color rgba="0.87 0.90 0.87 1.0"/>
-  </material>
-  <material name="Black">
-    <color rgba="0.08 0.08 0.08 1.0"/>
-  </material>
-  <material name="Gray">
-    <color rgba="0.2 0.2 0.21 1.0"/>
-  </material>
-  <material name="Green">
-    <color rgba="0.22 0.32 0.14 1.0"/>
-  </material>
-  <!--link name="arm_base_link"/-->
-  <joint name="arm_shoulder_pan_servo_joint" type="fixed">
-    <origin rpy="1.57079632679 0 1.57079632679" xyz="0 0 0"/>
-    <parent link="arm_base_link"/>
-    <child link="arm_shoulder_pan_servo_link"/>
-  </joint>
-  <link name="arm_shoulder_pan_servo_link">
-    <inertial>
-      <mass value="0.055"/>
-      <origin xyz="0 0 -0.01241"/>
-      <inertia ixx="1.80766666667e-05" ixy="0" ixz="0" iyy="1.82519791667e-05" iyz="0" izz="1.34119791667e-05"/>
-    </inertial>
-    <visual>
-      <origin rpy="0 0 0" xyz="0 0 0"/>
-      <geometry>
-        <mesh filename="package://pincher_arm_description/meshes/ax12_box.stl" scale="0.001 0.001 0.001"/>
-      </geometry>
-      <material name="Black"/>
-    </visual>
-    <collision>
-      <origin rpy="0 0 0" xyz="0.0 0.0 -0.01241"/>
-      <geometry>
-        <box size="0.0385 0.038 0.05"/>
-      </geometry>
-    </collision>
-  </link>
-  <gazebo reference="arm_shoulder_pan_servo_link">
-    <material>Gazebo/Black</material>
-    <selfCollide>true</selfCollide>
-    <gravity>true</gravity>
-  </gazebo>
-  <joint name="arm_shoulder_pan_joint" type="revolute">
-    <origin rpy="-1.57079632679 1.57079632679 3.14159265359" xyz="0 0.019 0"/>
-    <axis xyz="0 0 -1"/>
-    <limit effort="30" lower="-2.617" upper="2.617" velocity="1.571"/>
-    <dynamics friction="0.13"/>
-    <parent link="arm_shoulder_pan_servo_link"/>
-    <child link="arm_shoulder_pan_link"/>
-  </joint>
-  <link name="arm_shoulder_pan_link">
-    <inertial>
-      <mass value="0.008"/>
-      <origin xyz="0 0 0"/>
-      <inertia ixx="1.01666666667e-06" ixy="0" ixz="0" iyy="4.70666666667e-07" iyz="0" izz="1.37933333333e-06"/>
-    </inertial>
-    <visual>
-      <origin rpy="0 0 0" xyz="0 0 0"/>
-      <geometry>
-        <mesh filename="package://pincher_arm_description/meshes/F3.stl" scale="0.001 0.001 0.001"/>
-      </geometry>
-      <material name="Gray"/>
-    </visual>
-    <collision>
-      <origin rpy="0 0 0" xyz="0.0 0.0 -0.0045"/>
-      <geometry>
-        <box size="0.025 0.038 0.009"/>
-      </geometry>
-    </collision>
-  </link>
-  <gazebo reference="arm_shoulder_pan_link">
-    <material>Gazebo/Gray</material>
-    <selfCollide>true</selfCollide>
-    <gravity>true</gravity>
-  </gazebo>
-  <joint name="arm_shoulder_lift_servo_joint" type="fixed">
-    <origin rpy="0 3.14159265359 0" xyz="0 0 -0.0415"/>
-    <parent link="arm_shoulder_pan_link"/>
-    <child link="arm_shoulder_lift_servo_link"/>
-  </joint>
-  <link name="arm_shoulder_lift_servo_link">
-    <inertial>
-      <mass value="0.055"/>
-      <origin xyz="0 0 -0.01241"/>
-      <inertia ixx="1.80766666667e-05" ixy="0" ixz="0" iyy="1.82519791667e-05" iyz="0" izz="1.34119791667e-05"/>
-    </inertial>
-    <visual>
-      <origin rpy="0 0 0" xyz="0 0 0"/>
-      <geometry>
-        <mesh filename="package://pincher_arm_description/meshes/ax12_box.stl" scale="0.001 0.001 0.001"/>
-      </geometry>
-      <material name="Black"/>
-    </visual>
-    <collision>
-      <origin rpy="0 0 0" xyz="0.0 0.0 -0.01241"/>
-      <geometry>
-        <box size="0.0385 0.038 0.05"/>
-      </geometry>
-    </collision>
-  </link>
-  <gazebo reference="arm_shoulder_lift_servo_link">
-    <material>Gazebo/Black</material>
-    <selfCollide>true</selfCollide>
-    <gravity>true</gravity>
-  </gazebo>
-  <joint name="arm_shoulder_lift_joint" type="revolute">
-    <origin rpy="0 0 0" xyz="0 0 0"/>
-    <axis xyz="0 1 0"/>
-    <limit effort="30" lower="-2.09" upper="2.09" velocity="1.571"/>
-    <dynamics friction="0.13"/>
-    <parent link="arm_shoulder_lift_servo_link"/>
-    <child link="arm_shoulder_lift_link"/>
-  </joint>
-  <link name="arm_shoulder_lift_link">
-    <inertial>
-      <mass value="0.016"/>
-      <origin xyz="0 0 0"/>
-      <inertia ixx="8.76966666667e-06" ixy="0" ixz="0" iyy="6.67866666667e-06" iyz="0" izz="4.18166666667e-06"/>
-    </inertial>
-    <visual>
-      <origin rpy="0 0 0" xyz="0 0 0"/>
-      <geometry>
-        <mesh filename="package://pincher_arm_description/meshes/F4.stl" scale="0.001 0.001 0.001"/>
-      </geometry>
-      <material name="Gray"/>
-    </visual>
-    <collision>
-      <origin rpy="0 0 0" xyz="0.0 0.0 0.0215"/>
-      <geometry>
-        <box size="0.028 0.0485 0.065"/>
-      </geometry>
-    </collision>
-  </link>
-  <gazebo reference="arm_shoulder_lift_link">
-    <material>Gazebo/Gray</material>
-    <selfCollide>true</selfCollide>
-    <gravity>true</gravity>
-  </gazebo>
-  <joint name="arm_shoulder_F10_0_joint" type="fixed">
-    <origin rpy="0 0 0" xyz="0 0 0.0545"/>
-    <parent link="arm_shoulder_lift_link"/>
-    <child link="arm_shoulder_F10_0_link"/>
-  </joint>
-  <link name="arm_shoulder_F10_0_link">
-    <inertial>
-      <mass value="0.004"/>
-      <origin xyz="0 0 0"/>
-      <inertia ixx="4.86666666667e-07" ixy="0" ixz="0" iyy="2.13666666667e-07" iyz="0" izz="6.89666666667e-07"/>
-    </inertial>
-    <visual>
-      <origin rpy="0 0 0" xyz="0 0 0"/>
-      <geometry>
-        <mesh filename="package://pincher_arm_description/meshes/F10.stl" scale="0.001 0.001 0.001"/>
-      </geometry>
-      <material name="Gray"/>
-    </visual>
-    <collision>
-      <origin rpy="0 0 0" xyz="0.0 0.0 0.0"/>
-      <geometry>
-        <box size="0.025 0.038 0.004"/>
-      </geometry>
-    </collision>
-  </link>
-  <gazebo reference="arm_shoulder_F10_0_link">
-    <material>Gazebo/Gray</material>
-    <selfCollide>true</selfCollide>
-    <gravity>true</gravity>
-  </gazebo>
-  <joint name="arm_shoulder_F10_1_joint" type="fixed">
-    <origin rpy="0 0 0" xyz="0 0 0.004"/>
-    <parent link="arm_shoulder_F10_0_link"/>
-    <child link="arm_shoulder_F10_1_link"/>
-  </joint>
-  <link name="arm_shoulder_F10_1_link">
-    <inertial>
-      <mass value="0.004"/>
-      <origin xyz="0 0 0"/>
-      <inertia ixx="4.86666666667e-07" ixy="0" ixz="0" iyy="2.13666666667e-07" iyz="0" izz="6.89666666667e-07"/>
-    </inertial>
-    <visual>
-      <origin rpy="0 0 0" xyz="0 0 0"/>
-      <geometry>
-        <mesh filename="package://pincher_arm_description/meshes/F10.stl" scale="0.001 0.001 0.001"/>
-      </geometry>
-      <material name="Gray"/>
-    </visual>
-    <collision>
-      <origin rpy="0 0 0" xyz="0.0 0.0 0.0"/>
-      <geometry>
-        <box size="0.025 0.038 0.004"/>
-      </geometry>
-    </collision>
-  </link>
-  <gazebo reference="arm_shoulder_F10_1_link">
-    <material>Gazebo/Gray</material>
-    <selfCollide>true</selfCollide>
-    <gravity>true</gravity>
-  </gazebo>
-  <joint name="arm_shoulder_F10_2_joint" type="fixed">
-    <origin rpy="0 0 0" xyz="0 0 0.004"/>
-    <parent link="arm_shoulder_F10_1_link"/>
-    <child link="arm_shoulder_F10_2_link"/>
-  </joint>
-  <link name="arm_shoulder_F10_2_link">
-    <inertial>
-      <mass value="0.004"/>
-      <origin xyz="0 0 0"/>
-      <inertia ixx="4.86666666667e-07" ixy="0" ixz="0" iyy="2.13666666667e-07" iyz="0" izz="6.89666666667e-07"/>
-    </inertial>
-    <visual>
-      <origin rpy="0 0 0" xyz="0 0 0"/>
-      <geometry>
-        <mesh filename="package://pincher_arm_description/meshes/F10.stl" scale="0.001 0.001 0.001"/>
-      </geometry>
-      <material name="Gray"/>
-    </visual>
-    <collision>
-      <origin rpy="0 0 0" xyz="0.0 0.0 0.0"/>
-      <geometry>
-        <box size="0.025 0.038 0.004"/>
-      </geometry>
-    </collision>
-  </link>
-  <gazebo reference="arm_shoulder_F10_2_link">
-    <material>Gazebo/Gray</material>
-    <selfCollide>true</selfCollide>
-    <gravity>true</gravity>
-  </gazebo>
-  <joint name="arm_shoulder_F3_0_joint" type="fixed">
-    <origin rpy="0 3.14159265359 0" xyz="0 0 0.002"/>
-    <parent link="arm_shoulder_F10_2_link"/>
-    <child link="arm_shoulder_F3_0_link"/>
-  </joint>
-  <link name="arm_shoulder_F3_0_link">
-    <inertial>
-      <mass value="0.005"/>
-      <origin xyz="0 0 0"/>
-      <inertia ixx="6.35416666667e-07" ixy="0" ixz="0" iyy="2.94166666667e-07" iyz="0" izz="8.62083333333e-07"/>
-    </inertial>
-    <visual>
-      <origin rpy="0 0 0" xyz="0 0 0"/>
-      <geometry>
-        <mesh filename="package://pincher_arm_description/meshes/F3.stl" scale="0.001 0.001 0.001"/>
-      </geometry>
-      <material name="Gray"/>
-    </visual>
-    <collision>
-      <origin rpy="0 0 0" xyz="0.0 0.0 -0.0045"/>
-      <geometry>
-        <box size="0.025 0.038 0.009"/>
-      </geometry>
-    </collision>
-  </link>
-  <gazebo reference="arm_shoulder_F3_0_link">
-    <material>Gazebo/Gray</material>
-    <selfCollide>true</selfCollide>
-    <gravity>true</gravity>
-  </gazebo>
-  <joint name="arm_elbow_flex_servo_joint" type="fixed">
-    <origin rpy="0 3.14159265359 0" xyz="0 0 -0.0415"/>
-    <parent link="arm_shoulder_F3_0_link"/>
-    <child link="arm_elbow_flex_servo_link"/>
-  </joint>
-  <link name="arm_elbow_flex_servo_link">
-    <inertial>
-      <mass value="0.055"/>
-      <origin xyz="0 0 -0.01241"/>
-      <inertia ixx="1.80766666667e-05" ixy="0" ixz="0" iyy="1.82519791667e-05" iyz="0" izz="1.34119791667e-05"/>
-    </inertial>
-    <visual>
-      <origin rpy="0 0 0" xyz="0 0 0"/>
-      <geometry>
-        <mesh filename="package://pincher_arm_description/meshes/ax12_box.stl" scale="0.001 0.001 0.001"/>
-      </geometry>
-      <material name="Black"/>
-    </visual>
-    <collision>
-      <origin rpy="0 0 0" xyz="0.0 0.0 -0.01241"/>
-      <geometry>
-        <box size="0.0385 0.038 0.05"/>
-      </geometry>
-    </collision>
-  </link>
-  <gazebo reference="arm_elbow_flex_servo_link">
-    <material>Gazebo/Black</material>
-    <selfCollide>true</selfCollide>
-    <gravity>true</gravity>
-  </gazebo>
-  <joint name="arm_elbow_flex_joint" type="revolute">
-    <origin rpy="0 0 0" xyz="0 0 0"/>
-    <axis xyz="0 1 0"/>
-    <limit effort="30" lower="-2.42" upper="2.42" velocity="1.571"/>
-    <dynamics friction="0.13"/>
-    <parent link="arm_elbow_flex_servo_link"/>
-    <child link="arm_elbow_flex_link"/>
-  </joint>
-  <link name="arm_elbow_flex_link">
-    <inertial>
-      <mass value="0.016"/>
-      <origin xyz="0 0 0"/>
-      <inertia ixx="8.76966666667e-06" ixy="0" ixz="0" iyy="6.67866666667e-06" iyz="0" izz="4.18166666667e-06"/>
-    </inertial>
-    <visual>
-      <origin rpy="0 0 0" xyz="0 0 0"/>
-      <geometry>
-        <mesh filename="package://pincher_arm_description/meshes/F4.stl" scale="0.001 0.001 0.001"/>
-      </geometry>
-      <material name="Gray"/>
-    </visual>
-    <collision>
-      <origin rpy="0 0 0" xyz="0.0 0.0 0.0215"/>
-      <geometry>
-        <box size="0.028 0.0485 0.065"/>
-      </geometry>
-    </collision>
-  </link>
-  <gazebo reference="arm_elbow_flex_link">
-    <material>Gazebo/Gray</material>
-    <selfCollide>true</selfCollide>
-    <gravity>true</gravity>
-  </gazebo>
-  <joint name="arm_elbow_F10_0_joint" type="fixed">
-    <origin rpy="0 0 0" xyz="0 0 0.0545"/>
-    <parent link="arm_elbow_flex_link"/>
-    <child link="arm_elbow_F10_0_link"/>
-  </joint>
-  <link name="arm_elbow_F10_0_link">
-    <inertial>
-      <mass value="0.004"/>
-      <origin xyz="0 0 0"/>
-      <inertia ixx="4.86666666667e-07" ixy="0" ixz="0" iyy="2.13666666667e-07" iyz="0" izz="6.89666666667e-07"/>
-    </inertial>
-    <visual>
-      <origin rpy="0 0 0" xyz="0 0 0"/>
-      <geometry>
-        <mesh filename="package://pincher_arm_description/meshes/F10.stl" scale="0.001 0.001 0.001"/>
-      </geometry>
-      <material name="Gray"/>
-    </visual>
-    <collision>
-      <origin rpy="0 0 0" xyz="0.0 0.0 0.0"/>
-      <geometry>
-        <box size="0.025 0.038 0.004"/>
-      </geometry>
-    </collision>
-  </link>
-  <gazebo reference="arm_elbow_F10_0_link">
-    <material>Gazebo/Gray</material>
-    <selfCollide>true</selfCollide>
-    <gravity>true</gravity>
-  </gazebo>
-  <joint name="arm_elbow_F10_1_joint" type="fixed">
-    <origin rpy="0 0 0" xyz="0 0 0.004"/>
-    <parent link="arm_elbow_F10_0_link"/>
-    <child link="arm_elbow_F10_1_link"/>
-  </joint>
-  <link name="arm_elbow_F10_1_link">
-    <inertial>
-      <mass value="0.004"/>
-      <origin xyz="0 0 0"/>
-      <inertia ixx="4.86666666667e-07" ixy="0" ixz="0" iyy="2.13666666667e-07" iyz="0" izz="6.89666666667e-07"/>
-    </inertial>
-    <visual>
-      <origin rpy="0 0 0" xyz="0 0 0"/>
-      <geometry>
-        <mesh filename="package://pincher_arm_description/meshes/F10.stl" scale="0.001 0.001 0.001"/>
-      </geometry>
-      <material name="Gray"/>
-    </visual>
-    <collision>
-      <origin rpy="0 0 0" xyz="0.0 0.0 0.0"/>
-      <geometry>
-        <box size="0.025 0.038 0.004"/>
-      </geometry>
-    </collision>
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