Commit message: update urdf - Add manipulator

File: PC_user/src/Hardware/robotino/robotino_description/urdf/robotino.urdf (robot description, URDF)
Before this commit: robot robotino, 8 links, 7 joints
Links:
- removed link upper_platform_link
- added link AxisX_link; collision mesh filename=package://manipulator_description/meshes/AxisX.stl scale=0.001 0.001 0.001; visual mesh filename=package://manipulator_description/meshes/AxisX.stl scale=0.001 0.001 0.001
- added link AxisY_link; collision mesh filename=package://manipulator_description/meshes/AxisY.stl scale=0.001 0.001 0.001; visual mesh filename=package://manipulator_description/meshes/AxisY.stl scale=0.001 0.001 0.001
- added link AxisZ_link; collision mesh filename=package://manipulator_description/meshes/AxisZ.stl scale=0.001 0.001 0.001; visual mesh filename=package://manipulator_description/meshes/AxisZ.stl scale=0.001 0.001 0.001
- added link MovingPlate_link; collision mesh filename=package://manipulator_description/meshes/MovingPlate.stl scale=0.001 0.001 0.001; visual mesh filename=package://manipulator_description/meshes/MovingPlate.stl scale=0.001 0.001 0.001
- added link tower_link; collision mesh filename=package://robotino_description/model/Robotino3_Platform.dae scale=0.009 0.009 0.009; visual mesh filename=package://robotino_description/model/Robotino3_Platform.dae scale=0.009 0.009 0.009
- link base_link: geometry collision mesh filename=package://robotino_description/model/Robotino3_SplitMain_No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 scale=0.01 0.01 0.01; visual mesh filename=package://robotino_description/model/Robotino3_SplitMain_No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 scale=0.01 0.01 0.01
- link platform_link: geometry 
Joints:
- removed joint base_to_kinect
- removed joint upper_platform_joint
- added joint AxisX_joint: type fixed, parent platform_link, child AxisX_link, origin xyz=0.160 -0.115 0.0015 rpy=0 0 1.570796
- added joint AxisY_joint: type prismatic, parent AxisX_link, child AxisY_link, origin xyz=-0.01 0.308 0.0225 rpy=1.5708 0 0, axis 0 0 1, limit lower=0 upper=0.234 effort=0.1 velocity=0.1
- added joint AxisZ_joint: type prismatic, parent AxisY_link, child AxisZ_link, origin xyz=0.039 0.08 0.006 rpy=-1.5708 0 0, axis 1 0 0, limit lower=0 upper=0.105 effort=0.1 velocity=0.1
- added joint MovingPlate_joint: type prismatic, parent AxisZ_link, child MovingPlate_link, origin xyz=-0.032 -0.076 0.38 rpy=-1.5708 3.1415 0, axis 0 1 0, limit lower=0 upper=0.18 effort=0.1 velocity=0.1
- added joint platform_to_kinect: type fixed, parent platform_link, child camera_link, origin xyz= 0.17 0 0.025 rpy=0 0.35 0
- added joint tower_joint: type fixed, parent base_link, child tower_link, origin xyz=0 0 0.06 rpy=0 0 1.5707, axis 0 0 0
- joint platform_joint: axis 0 0 0 -> (none); origin xyz=0 0 0.06 rpy=0 0 0 -> xyz=0 0 0.76 rpy=0 0 0
- joint wheel0_joint: origin xyz=-0.0001 0.1825 0.059154 rpy=0 0 0 -> xyz=-0.1825 -0.0001 0.059154 rpy=0 0 1.570796
- joint wheel1_joint: origin xyz=-0.157067 -0.090625 0.059154 rpy=0 0 2.094395102393195 -> xyz=0.090625 -0.157067 0.059154 rpy=0 0 3.665191
- joint wheel2_joint: origin xyz=0.156867 -0.090625 0.059154 rpy=0 0 -2.094395102393195 -> xyz=0.090625 0.156867 0.059154 rpy=0 0 -0.523599
