Commit message: Vacaciones

File: PC_user/src/Hardware/justina/justina_description/urdf/justina_left_arm.xacro (robot description, xacro)
@@ -13,7 +13,7 @@
     </visual>
     <collision>
-      <origin xyz="0 -0.01 0.02" rpy = "0 0 0"/>
-      <geometry>
-        <box size = "0.04025 0.108 0.065"/>
+      <origin xyz="0 -0.01 0.02" rpy = "0 3.1415 0"/>
+      <geometry>
+        <mesh filename="package://justina_description/stl/servos/Mx106-2.dae"/>
       </geometry>
     </collision>
@@ -37,11 +37,11 @@
     </visual>
     <collision>
-      <origin xyz="0 -0.01 -0.04881" rpy = "0 0 0"/>
-      <geometry>
-        <box size = "0.04025 0.06 0.04025"/>
-      </geometry>
-    </collision>
-    <inertial>
-      <origin xyz="0 -0.01 -0.04881" rpy = "0 0 0"/>
+      <origin xyz="0 -0.01 0.0" rpy = "0 0 -1.5707"/>
+      <geometry>
+        <mesh filename="package://justina_description/stl/servos/Mx106-s.dae"/>
+      </geometry>
+    </collision>
+    <inertial>
+      <origin xyz="0 -0.01 0.0" rpy = "0 0 -1.5707"/>
       <mass value="0.125"/>
       <inertia
@@ -69,13 +69,13 @@
     </visual>
     <collision>
-      <origin xyz="0 0 -0.125" rpy = "0 0 0"/>
-      <geometry>
-        <box size = "0.04025 0.04025 0.19"/>
-      </geometry>
-    </collision>
-    <collision>
-      <origin xyz="-0.01 0 -0.197" rpy = "0 0 0"/>
-      <geometry>
-        <box size = "0.06 0.04025 0.04025"/>
+      <origin xyz="0 0 -0.00125" rpy = "0 0 0"/>
+      <geometry>
+        <mesh filename="package://justina_description/stl/arm/bone_1.dae"/>
+      </geometry>
+    </collision>
+    <collision>
+      <origin xyz="-0.0 0 -0.197" rpy = "0 0 -1.5707"/>
+      <geometry>
+        <mesh filename="package://justina_description/stl/servos/Mx64.dae"/>
       </geometry>
     </collision>
@@ -99,11 +99,11 @@
     </visual>
     <collision>
-      <origin xyz="0 0 -0.04" rpy = "0 0 0"/>
-      <geometry>
-        <box size = "0.04025 0.04025 0.06"/>
-      </geometry>
-    </collision>
-    <inertial>
-      <origin xyz="0 0 -0.04" rpy = "0 0 0"/>
+      <origin xyz="0.012 0.0 -0.025" rpy = "0 1.5707 -1.5707"/>
+      <geometry>
+          <mesh filename="package://justina_description/stl/servos/Mx64.dae"/>
+      </geometry>
+    </collision>
+    <inertial>
+      <origin xyz="0.012 0.0 -0.025" rpy = "0 1.5707 -1.5707"/>
       <mass value="0.125"/>
       <inertia
@@ -131,13 +131,13 @@
     </visual>
     <collision>
-      <origin xyz="0 0 -0.11" rpy = "0 0 0"/>
-      <geometry>
-        <box size = "0.04025 0.04025 0.16"/>
-      </geometry>
-    </collision>
-    <collision>
-      <origin xyz="-0.01 0 -0.167" rpy = "0 0 0"/>
-      <geometry>
-        <box size = "0.06 0.04025 0.04025"/>
+      <origin xyz="0 0 -0.0" rpy = "0 0 0"/>
+      <geometry>
+        <mesh filename="package://justina_description/stl/arm/bone_2.dae"/>
+      </geometry>
+    </collision>
+    <collision>
+      <origin xyz="-0.0 0 -0.168" rpy = "0 0 3.1415"/>
+      <geometry>
+        <mesh filename="package://justina_description/stl/servos/Mx64.dae"/>
       </geometry>
     </collision>
@@ -161,11 +161,11 @@
     </visual>
     <collision>
+      <origin xyz="0 0 -0.03" rpy = "0 1.5707 -1.5707"/>
+      <geometry>
+        <mesh filename="package://justina_description/stl/servos/Mx64.dae"/>
+      </geometry>
+    </collision>
+    <inertial>
       <origin xyz="0 0 -0.025" rpy = "0 0 0"/>
-      <geometry>
-        <box size = "0.04025 0.04025 0.02"/>
-      </geometry>
-    </collision>
-    <inertial>
-      <origin xyz="0 0 -0.025" rpy = "0 0 0"/>
       <mass value="0.125"/>
       <inertia
@@ -184,7 +184,7 @@
     </visual>
     <collision>
-      <origin xyz="0 0 -0.042" rpy = "0 0 0"/>
-      <geometry>
-        <box size = "0.04025 0.04025 0.04"/>
+      <origin xyz="0 0 -0.052" rpy = "0 0 0"/>
+      <geometry>
+        <mesh filename="package://justina_description/stl/servos/Mx64.dae"/>
       </geometry>
     </collision>
@@ -214,9 +214,10 @@
     </visual>
     <collision>
-      <origin xyz="-0.01 0 -0.03" rpy = "0 0 0"/>
-      <geometry>
-        <box size = "0.06 0.03525 0.03525"/>
-      </geometry>
-    </collision>
+      <origin xyz="0 0 -0.055" rpy = "1.5707 1.5707 0"/>
+      <geometry>
+        <mesh filename="package://justina_description/stl/servos/Mx28-2.dae"/>
+      </geometry>
+    </collision>
+    <!--
     <collision>
       <origin xyz="0 0 -0.055" rpy = "0 0 0"/>
@@ -225,4 +226,5 @@
       </geometry>
     </collision>
+    -->
     <inertial>
       <origin xyz="-0.01 0 -0.05" rpy = "0 0 0"/>
@@ -244,7 +246,7 @@
     </visual>
     <collision>
-      <origin xyz="0 0 -0.065" rpy = "0 0 0"/>
-      <geometry>
-        <box size = "0.04 0.005 0.09"/>
+      <origin xyz="0 0 0.0" rpy = "0 1.5707 0"/>
+      <geometry>
+          <mesh filename="package://justina_description/stl/arm/gripper.dae"/>
       </geometry>
     </collision>
@@ -268,7 +270,7 @@
     </visual>
     <collision>
-      <origin xyz="0 0 -0.065" rpy = "0 0 0"/>
-      <geometry>
-        <box size = "0.04 0.005 0.09"/>
+      <origin xyz="0 0 -0.0" rpy = "0 1.5707 3.1415"/>
+      <geometry>
+        <mesh filename="package://justina_description/stl/arm/gripper.dae"/>
       </geometry>
     </collision>

File: PC_user/src/Hardware/robotino/robotino_description/urdf/jestino_base.urdf.xacro (robot description, xacro)
@@ -44,6 +44,6 @@
   <!-- ***************************** Tower ******************************************* -->
 <link name="tower_link">
+  <!-- aluminium axis -->
   <visual>
-    <!-- Caja (torre principal) -->
     <origin xyz="0 0 0.41" rpy="0 0 0"/>
     <geometry>
@@ -55,5 +55,4 @@
   </visual>
   <visual>
-    <!-- Cilindro encima de la caja -->
     <origin xyz="0 0 0.705" rpy="0 0 0"/>
     <geometry>
@@ -62,6 +61,6 @@
     <material name="aluminium"/>
   </visual>
+  <!-- aluminium axis -->
   <collision>
-    <!-- Caja -->
     <origin xyz="0 0 0.41" rpy="0 0 0"/>
     <geometry>
@@ -70,8 +69,14 @@
   </collision>
   <collision>
-    <!-- Cilindro -->
     <origin xyz="0 0 0.705" rpy="0 0 0"/>
     <geometry>
       <cylinder radius="0.075" length="0.005"/>
+    </geometry>
+  </collision>
+  <!-- Laptop -->
+  <collision>
+    <origin xyz="-0.04 0.0 0.30" rpy="0 0 0"/>
+    <geometry>
+      <box size = "0.03 0.35 0.20"/>
     </geometry>
   </collision>
@@ -97,4 +102,10 @@
       <origin xyz="0 0 -0.055" rpy="0 0 1.57"/>
     </visual>
+    <collision>
+      <geometry>
+        <mesh filename="package://robotino_description/meshes/sensors/hokuyo.dae" scale="0.01 0.01 0.01"/>
+      </geometry>
+      <origin xyz="0 0 -0.055" rpy="0 0 1.57"/>
+    </collision>
   </link>
   <joint name="base_to_hokuyo" type="fixed">
