Commit message: change left arm xacro

File: PC_user/src/Hardware/justina/justina_description/urdf/justina.xacro (robot description, xacro)
@@ -5,5 +5,5 @@
   <xacro:include filename="$(find robotino_description)/urdf/jestino_base.urdf.xacro"/>
   <xacro:include filename="$(find justina_description)/urdf/justina_torso.xacro"/>
-  <!--xacro:include filename="$(find justina_description)/urdf/justina_left_arm.xacro"/-->
+  <xacro:include filename="$(find justina_description)/urdf/justina_left_arm.xacro"/>
   <!--xacro:include filename="$(find justina_description)/urdf/justina_right_arm.xacro"/-->
   <xacro:include filename="$(find justina_description)/urdf/justina_head.xacro"/>

File: PC_user/src/Hardware/justina/justina_description/urdf/justina_left_arm.xacro (robot description, xacro)
@@ -91,5 +91,5 @@
   <link name="left_arm_link3">
     <visual>
-      <origin xyz="0.012 0.0 -0.025" rpy = "0 1.5707 -1.5707"/>
+      <origin xyz="-0.0 0.0 -0.075" rpy = "1.5707 -3.1425 0"/>
       <geometry>
         <!--box size = "0.04025 0.04025 0.06"/-->
@@ -105,5 +105,5 @@
     </collision>
     <inertial>
-      <origin xyz="0.012 0.0 -0.025" rpy = "0 1.5707 -1.5707"/>
+      <origin xyz="-0.0 0.0 -0.075" rpy = "1.5707 -3.1425 0"/>
       <mass value="0.125"/>
       <inertia
@@ -115,5 +115,5 @@
   <link name="left_arm_link4">
     <visual>
-      <origin xyz="0 0 -0.0" rpy = "0 0 0"/>
+      <origin xyz="0 -0.0025 -0.0" rpy = "0 0 0"/>
       <geometry>
         <mesh filename="package://justina_description/stl/arm/bone_2.dae"/>
@@ -123,5 +123,5 @@
     </visual>
     <visual>
-      <origin xyz="-0.0 0 -0.168" rpy = "0 0 3.1415"/>
+      <origin xyz="-0.0 0 -0.16" rpy = "0 0 -1.5707"/>
       <geometry>
         <!--box size = "0.06 0.04025 0.04025"/-->
@@ -131,5 +131,5 @@
     </visual>
     <collision>
-      <origin xyz="0 0 -0.0" rpy = "0 0 0"/>
+      <origin xyz="0 0.0025 -0.0" rpy = "0 0 0"/>
       <geometry>
         <mesh filename="package://justina_description/stl/arm/bone_2.dae"/>
@@ -137,5 +137,5 @@
     </collision>
     <collision>
-      <origin xyz="-0.0 0 -0.168" rpy = "0 0 3.1415"/>
+      <origin xyz="-0.0 0 -0.16" rpy = "0 0 -1.5707"/>
       <geometry>
         <mesh filename="package://justina_description/stl/servos/Mx64.dae"/>
@@ -153,5 +153,5 @@
   <link name="left_arm_link5">
     <visual>
-      <origin xyz="0 0 -0.03" rpy = "0 1.5707 -1.5707"/>
+      <origin xyz="0 0 -0.05" rpy = "1.5707 0 0"/>
       <geometry>
         <!--box size = "0.04025 0.04025 0.02"/-->
@@ -161,5 +161,5 @@
     </visual>
     <collision>
-      <origin xyz="0 0 -0.03" rpy = "0 1.5707 -1.5707"/>
+      <origin xyz="0 0 -0.05" rpy = "1.5707 0 0"/>
       <geometry>
         <mesh filename="package://justina_description/stl/servos/Mx64.dae"/>
@@ -177,18 +177,18 @@
   <link name="left_arm_link6">
     <visual>
-      <origin xyz="0 0 -0.052" rpy = "0 0 0"/>
-      <geometry>
-        <mesh filename="package://justina_description/stl/servos/Mx64.dae"/>
-      </geometry>
-      <material name = "la_material"><color rgba="1.0 0.5 0 1"/></material>
-    </visual>
-    <collision>
-      <origin xyz="0 0 -0.052" rpy = "0 0 0"/>
-      <geometry>
-        <mesh filename="package://justina_description/stl/servos/Mx64.dae"/>
-      </geometry>
-    </collision>
-    <inertial>
-      <origin xyz="0 0 -0.042" rpy = "0 0 0"/>
+      <origin xyz="0 0 -0.08" rpy = "0 0 -1.5707"/>
+      <geometry>
+        <mesh filename="package://justina_description/stl/servos/Mx64.dae"/>
+      </geometry>
+      <material name = "la_material"><color rgba="1.0 0.5 0 1"/></material>
+    </visual>
+    <collision>
+      <origin xyz="0 0 -0.08" rpy = "0 0 0"/>
+      <geometry>
+        <mesh filename="package://justina_description/stl/servos/Mx64.dae"/>
+      </geometry>
+    </collision>
+    <inertial>
+      <origin xyz="0 0 -0.042" rpy = "0 0 1.5707"/>
       <mass value="0.125"/>
       <inertia
@@ -302,5 +302,5 @@
   </joint>
   <joint name="la_3_joint" type="revolute">
-    <origin xyz="0 0 -0.215" rpy="0 0 0"/>
+    <origin xyz="0 0 -0.195" rpy="0 0 0"/>
     <parent link="left_arm_link2"/>
     <child link="left_arm_link3"/>
@@ -310,5 +310,5 @@
   </joint>
   <joint name="la_4_joint" type="revolute">
-    <origin xyz="0.015 0 -0.025" rpy="0 0 0"/>
+    <origin xyz="0.0 0 -0.070" rpy="0 0 0"/>
     <parent link="left_arm_link3"/>
     <child link="left_arm_link4"/>
@@ -318,5 +318,5 @@
   </joint>
   <joint name="la_5_joint" type="revolute">
-    <origin xyz="0 0 -0.183" rpy="0 0 0"/>
+    <origin xyz="0 0 -0.16" rpy="0 0 0"/>
     <parent link="left_arm_link4"/>
     <child link="left_arm_link5"/>
@@ -326,5 +326,5 @@
   </joint>
   <joint name="la_6_joint" type="revolute">
-    <origin xyz="0 0.0 -0.03" rpy="0 0 0"/>
+    <origin xyz="0 0.0 -0.05" rpy="0 0 0"/>
     <parent link="left_arm_link5"/>
     <child link="left_arm_link6"/>
@@ -334,5 +334,5 @@
   </joint>
   <joint name="la_7_joint" type="revolute">
-    <origin xyz="0 0.0 -0.055" rpy="0 0 0"/>
+    <origin xyz="0 0.0 -0.08" rpy="0 0 0"/>
     <parent link="left_arm_link6"/>
     <child link="left_arm_link7"/>
